File: kicad/wireless-pcb/accelerometer.kicad_sch (KiCad schematic)
At the start: 5 parts, among them U2 ADXL363

Commit message: Various cleanup, better pin selection, etc.
Parts:
- U2: value ADXL363 -> ADXL362; LCSC (none) -> C192252
Changed lines of the file:
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@@
       (effects (font (size 1.27 1.27)))
     )
-    (property "Value" "ADXL363" (at 127 71.3039 0)
+    (property "Value" "ADXL362" (at 127 71.3039 0)
       (effects (font (size 1.27 1.27)))
     )
@@
       (effects (font (size 1.27 1.27)) hide)
     )
+    (property "LCSC" "C192252" (at 111.76 75.692 0)
+      (effects (font (size 1.27 1.27)) hide)
+    )

Commit message: BOM tweaks, add some test points, minor placement tweaks.
Parts:
- U2: MPN (none) -> ADXL362BCCZ-RL7
Changed lines of the file:
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@@
+      (effects (font (size 1.27 1.27)) hide)
+    )
+    (property "MPN" "ADXL362BCCZ-RL7" (at 111.76 75.692 0)
       (effects (font (size 1.27 1.27)) hide)
     )
