File: kicad/wireless-pcb/analog.kicad_sch (KiCad schematic)
At the start: 20 parts, among them U2 74HC4051, U5 OPA357AIDBVR

Commit message: BOM tweaks, add some test points, minor placement tweaks.
Parts:
- U2: MPN (none) -> 74HC4051PW,118
- U5: MPN (none) -> OPA357AIDBVR
Changed lines of the file:
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@@
+      (effects (font (size 1.27 1.27)) hide)
+    )
+    (property "MPN" "OPA357AIDBVR" (at 190.246 84.582 0)
       (effects (font (size 1.27 1.27)) hide)
     )
@@
     )
     (property "JlcRotOffset" "90" (at 105.156 49.53 0)
+      (effects (font (size 1.27 1.27)) hide)
+    )
+    (property "MPN" "74HC4051PW,118" (at 105.156 49.53 0)
       (effects (font (size 1.27 1.27)) hide)
     )
@@
       (effects (font (size 1.27 1.27)) hide)
     )
+    (property "MPN" "74HC4051PW,118" (at 104.14 115.062 0)
+      (effects (font (size 1.27 1.27)) hide)
+    )
